File: Hardware/Release Design Files/Source Kicad Files/SwitchBlox.sch (KiCad schematic (older format))
At the start: 16 parts, among them J1 CONN_HEADER_V_5, J2 CONN_HEADER_V_5, J3 CONN_HEADER_V_5, J4 CONN_HEADER_V_5, J5 CONN_HEADER_V_5, J6 CONN_HEADER_V_5, J7 CONN_HEADER_V_5, J8 Conn_02x06_Odd_Even, SW1 SW_Push, U1 RevTable

Commit message: Restructured files, added logo.
Other:
- note added: "OPEN SOURCE HARDWARE\n"
- note added: "Released under Creative Commons - Attribution - ShareAlike 3.0"
- note added: "SwitchBlox Rev B\n"
- note removed: "SwitchBlox"
